Commit message: Can do some SLAM now

File: description/sage.urdf.xacro (robot description, xacro)
@@ -2,11 +2,11 @@
 <robot xmlns:xacro="http://www.ros.org/wiki/xacro" name="sage">
   <!-- === Dimensions === -->
-  <xacro:property name="base_length" value="0.50"/>
-  <xacro:property name="base_width" value="0.50"/>
+  <xacro:property name="base_width" value="0.3691"/>
+  <xacro:property name="base_length" value="0.4083"/>
   <xacro:property name="base_thickness" value="0.02"/>
-  <xacro:property name="wheel_radius" value="0.06"/>
-  <xacro:property name="wheel_thickness" value="0.035"/>
-  <xacro:property name="wheel_x_from_back" value="0.10"/>
-  <xacro:property name="lidar_height" value="0.20"/>
+  <xacro:property name="wheel_radius" value="0.0505"/>
+  <xacro:property name="wheel_thickness" value="0.0254"/>
+  <xacro:property name="wheel_x_from_back" value="0.0658"/>
+  <xacro:property name="lidar_height" value="0.2124"/>
   <xacro:property name="base_z" value="${wheel_radius}"/>
   <xacro:property name="half_len" value="${base_length/2.0}"/>
@@ -112,5 +112,5 @@
     <parent link="base_link"/>
     <child link="lidar_link"/>
-    <origin xyz="0 0 ${lidar_height}" rpy="0 0 0"/>
+    <origin xyz="0 0 ${lidar_height}" rpy="0 0 ${pi}"/> <!-- LIDAR mounted 180 degrees rotated I think -->
   </joint>
   <!-- === Nav2 footprint (optional) === -->

Commit message: updated some configs

File: description/sage.urdf.xacro (robot description, xacro)
@@ -6,11 +6,13 @@
   <xacro:property name="base_thickness" value="0.02"/>
   <xacro:property name="wheel_radius" value="0.0505"/>
+  <xacro:property name="front_wheel_radius" value="0.0415"/>
   <xacro:property name="wheel_thickness" value="0.0254"/>
   <xacro:property name="wheel_x_from_back" value="0.0658"/>
+  <xacro:property name="front_wheel_x_from_front" value="0.04572"/>
   <xacro:property name="lidar_height" value="0.2124"/>
-  <xacro:property name="base_z" value="${wheel_radius}"/>
+  <xacro:property name="base_z" value="0.08731"/>
   <xacro:property name="half_len" value="${base_length/2.0}"/>
   <xacro:property name="half_wid" value="${base_width/2.0}"/>
-  <xacro:property name="track_width" value="${base_width + wheel_thickness}"/>
+  <xacro:property name="track_width" value="0.4953"/>
   <xacro:property name="half_track" value="${track_width / 2.0}"/>
   <xacro:property name="rear_wheel_x" value="${-half_len + wheel_x_from_back}"/>
@@ -76,5 +78,5 @@
         <origin xyz="0 0 0" rpy="${pi/2} 0 0"/>
         <geometry>
-          <cylinder radius="${wheel_radius * 0.5}" length="${wheel_thickness}"/>
+          <cylinder radius="${front_wheel_radius}" length="${wheel_thickness}"/>
         </geometry>
         <material name="black"/>
@@ -83,5 +85,5 @@
         <origin xyz="0 0 0" rpy="${pi/2} 0 0"/>
         <geometry>
-          <cylinder radius="${wheel_radius * 0.5}" length="${wheel_thickness}"/>
+          <cylinder radius="${front_wheel_radius}" length="${wheel_thickness}"/>
         </geometry>
       </collision>
@@ -94,5 +96,5 @@
       <parent link="base_link"/>
       <child link="${name}"/>
-      <origin xyz="${half_len - 0.08} ${y} ${wheel_radius}" rpy="0 0 0"/>
+      <origin xyz="${half_len - front_wheel_x_from_front} ${y} ${wheel_radius}" rpy="0 0 0"/>
     </joint>
   </xacro:macro>

Commit message: serial communication setup between MCU and jetson, with update protocol to take care of IMU and wheel odom

File: description/sage.urdf.xacro (robot description, xacro)
@@ -116,4 +116,29 @@
     <origin xyz="0 0 ${lidar_height}" rpy="0 0 ${pi}"/> <!-- LIDAR mounted 180 degrees rotated I think -->
   </joint>
+  <!-- === IMU Link === -->
+  <link name="imu_link">
+    <visual>
+      <origin xyz="0 0 0" rpy="0 0 0"/>
+      <geometry>
+        <box size="0.03 0.03 0.01"/> <!-- Example dimensions for the IMU -->
+      </geometry>
+      <material name="blue"/>
+    </visual>
+    <collision>
+      <origin xyz="0 0 0" rpy="0 0 0"/>
+      <geometry>
+        <box size="0.03 0.03 0.01"/>
+      </geometry>
+    </collision>
+    <inertial>
+      <mass value="0.05"/> <!-- Example mass for the IMU -->
+      <inertia ixx="0.0001" ixy="0" ixz="0" iyy="0.0001" iyz="0" izz="0.0001"/>
+    </inertial>
+  </link>
+  <joint name="imu_mount" type="fixed">
+    <parent link="base_link"/>
+    <child link="imu_link"/>
+    <origin xyz="0.085725 -0.0635 ${base_z + base_thickness/2.0}" rpy="0 ${pi/2} 0"/> <!-- Corrected z-coordinate -->
+  </joint>
   <!-- === Nav2 footprint (optional) === -->
   <link name="base_footprint"/>

Commit message: mapped gellersen and localization working well

File: description/sage.urdf.xacro (robot description, xacro)
@@ -116,29 +116,4 @@
     <origin xyz="0 0 ${lidar_height}" rpy="0 0 ${pi}"/> <!-- LIDAR mounted 180 degrees rotated I think -->
   </joint>
-  <!-- === IMU Link === -->
-  <link name="imu_link">
-    <visual>
-      <origin xyz="0 0 0" rpy="0 0 0"/>
-      <geometry>
-        <box size="0.03 0.03 0.01"/> <!-- Example dimensions for the IMU -->
-      </geometry>
-      <material name="blue"/>
-    </visual>
-    <collision>
-      <origin xyz="0 0 0" rpy="0 0 0"/>
-      <geometry>
-        <box size="0.03 0.03 0.01"/>
-      </geometry>
-    </collision>
-    <inertial>
-      <mass value="0.05"/> <!-- Example mass for the IMU -->
-      <inertia ixx="0.0001" ixy="0" ixz="0" iyy="0.0001" iyz="0" izz="0.0001"/>
-    </inertial>
-  </link>
-  <joint name="imu_mount" type="fixed">
-    <parent link="base_link"/>
-    <child link="imu_link"/>
-    <origin xyz="0.085725 -0.0635 ${base_z + base_thickness/2.0}" rpy="0 ${pi/2} 0"/> <!-- Corrected z-coordinate -->
-  </joint>
   <!-- === Nav2 footprint (optional) === -->
   <link name="base_footprint"/>

Commit message: updated runs without imu and change robot description to adjust for new lid

File: description/sage.urdf.xacro (robot description, xacro)
@@ -2,17 +2,17 @@
 <robot xmlns:xacro="http://www.ros.org/wiki/xacro" name="sage">
   <!-- === Dimensions === -->
-  <xacro:property name="base_width" value="0.3691"/>
-  <xacro:property name="base_length" value="0.4083"/>
-  <xacro:property name="base_thickness" value="0.02"/>
-  <xacro:property name="wheel_radius" value="0.0505"/>
-  <xacro:property name="front_wheel_radius" value="0.0415"/>
-  <xacro:property name="wheel_thickness" value="0.0254"/>
-  <xacro:property name="wheel_x_from_back" value="0.0658"/>
-  <xacro:property name="front_wheel_x_from_front" value="0.04572"/>
-  <xacro:property name="lidar_height" value="0.2124"/>
-  <xacro:property name="base_z" value="0.08731"/>
+  <xacro:property name="base_width" value="0.3048"/>
+  <xacro:property name="base_length" value="0.558"/>
+  <xacro:property name="base_thickness" value="0.043"/>
+  <xacro:property name="wheel_radius" value="0.0762"/>
+  <xacro:property name="front_wheel_radius" value="0.0762"/>
+  <xacro:property name="wheel_thickness" value="0.0508"/>
+  <xacro:property name="wheel_x_from_back" value="0.04608"/>
+  <xacro:property name="front_wheel_x_from_front" value="0.044718"/>
+  <xacro:property name="lidar_height" value="0.5268"/>
+  <xacro:property name="base_z" value="0.0522"/>
   <xacro:property name="half_len" value="${base_length/2.0}"/>
   <xacro:property name="half_wid" value="${base_width/2.0}"/>
-  <xacro:property name="track_width" value="0.4953"/>
+  <xacro:property name="track_width" value="0.3612"/>
   <xacro:property name="half_track" value="${track_width / 2.0}"/>
   <xacro:property name="rear_wheel_x" value="${-half_len + wheel_x_from_back}"/>
@@ -29,5 +29,5 @@
     </inertial>
     <visual>
-      <origin xyz="0 0 ${base_z + base_thickness/2.0}" rpy="0 0 0"/>
+      <origin xyz="0 0 ${base_z + base_thickness}" rpy="0 0 0"/>
       <geometry>
         <box size="${base_length} ${base_width} ${base_thickness}"/>
@@ -36,5 +36,5 @@
     </visual>
     <collision>
-      <origin xyz="0 0 ${base_z + base_thickness/2.0}" rpy="0 0 0"/>
+      <origin xyz="0 0 ${base_z + base_thickness}" rpy="0 0 0"/>
       <geometry>
         <box size="${base_length} ${base_width} ${base_thickness}"/>
@@ -114,5 +114,31 @@
     <parent link="base_link"/>
     <child link="lidar_link"/>
-    <origin xyz="0 0 ${lidar_height}" rpy="0 0 ${pi}"/> <!-- LIDAR mounted 180 degrees rotated I think -->
+    <!-- <origin xyz="0 0 ${lidar_height}" rpy="0 0 ${pi}"/>  LIDAR mounted 180 degrees rotated I think -->
+    <origin xyz="-0.1466 0 ${lidar_height}" rpy="0 0 0"/> <!-- LIDAR mounted 180 degrees rotated I think. Its moved -146.6mm from center -->
+  </joint>
+  <!-- === IMU Link === -->
+  <link name="imu_link">
+    <visual>
+      <origin xyz="0 0 0" rpy="0 0 0"/>
+      <geometry>
+        <box size="0.03 0.03 0.01"/> <!-- Example dimensions for the IMU -->
+      </geometry>
+      <material name="blue"/>
+    </visual>
+    <collision>
+      <origin xyz="0 0 0" rpy="0 0 0"/>
+      <geometry>
+        <box size="0.03 0.03 0.01"/>
+      </geometry>
+    </collision>
+    <inertial>
+      <mass value="0.05"/> <!-- Example mass for the IMU -->
+      <inertia ixx="0.0001" ixy="0" ixz="0" iyy="0.0001" iyz="0" izz="0.0001"/>
+    </inertial>
+  </link>
+  <joint name="imu_mount" type="fixed">
+    <parent link="base_link"/>
+    <child link="imu_link"/>
+    <origin xyz="0.09756 -0.102 ${base_z + base_thickness}" rpy="0 ${pi/2} 0"/> <!-- Corrected z-coordinate -->
   </joint>
   <!-- === Nav2 footprint (optional) === -->

File: description/sagewithoutimu.urdf.xacro (robot description, xacro)
@@ -115,30 +115,5 @@
     <child link="lidar_link"/>
     <!-- <origin xyz="0 0 ${lidar_height}" rpy="0 0 ${pi}"/>  LIDAR mounted 180 degrees rotated I think -->
-    <origin xyz="0 0 ${lidar_height}" rpy="0 0 0"/> <!-- LIDAR mounted 180 degrees rotated I think -->
-  </joint>
-  <!-- === IMU Link === -->
-  <link name="imu_link">
-    <visual>
-      <origin xyz="0 0 0" rpy="0 0 0"/>
-      <geometry>
-        <box size="0.03 0.03 0.01"/> <!-- Example dimensions for the IMU -->
-      </geometry>
-      <material name="blue"/>
-    </visual>
-    <collision>
-      <origin xyz="0 0 0" rpy="0 0 0"/>
-      <geometry>
-        <box size="0.03 0.03 0.01"/>
-      </geometry>
-    </collision>
-    <inertial>
-      <mass value="0.05"/> <!-- Example mass for the IMU -->
-      <inertia ixx="0.0001" ixy="0" ixz="0" iyy="0.0001" iyz="0" izz="0.0001"/>
-    </inertial>
-  </link>
-  <joint name="imu_mount" type="fixed">
-    <parent link="base_link"/>
-    <child link="imu_link"/>
-    <origin xyz="0.09756 -0.102 ${base_z + base_thickness}" rpy="0 ${pi/2} 0"/> <!-- Corrected z-coordinate -->
+    <origin xyz="-0.1466 0 ${lidar_height}" rpy="0 0 0"/> <!-- LIDAR mounted 180 degrees rotated I think. Its moved -146.6mm from center-->
   </joint>
   <!-- === Nav2 footprint (optional) === -->

Commit message: Deployment ready state

File: description/sage.urdf.xacro (robot description, xacro)
@@ -142,4 +142,19 @@
     <origin xyz="0.09756 -0.102 ${base_z + base_thickness}" rpy="0 ${pi/2} 0"/> <!-- Corrected z-coordinate -->
   </joint>
+<!-- === Camera Link === -->
+  <link name="camera_link">
+    <visual>
+      <origin xyz="0 0 0" rpy="0 0 0"/>
+      <geometry>
+        <cylinder radius="0.03" length="0.05"/>
+      </geometry>
+      <material name="black"/>
+    </visual>
+  </link>
+  <joint name="camera_joint" type="fixed">
+    <parent link="base_link"/>
+    <child link="camera_link"/>
+    <origin xyz="0.179 0.017 0.523" rpy="-1.5707963 0 -1.5707963"/>
+  </joint>
   <!-- === Nav2 footprint (optional) === -->
   <link name="base_footprint"/>
